Commit message: asset conversion

File: assets/allegro/allegro.urdf (robot description, URDF)
Before this commit: robot allegro_hand_right, 21 links, 20 joints
Links:
- removed link link_0.0
- removed link link_1.0
- removed link link_10.0
- removed link link_11.0
- removed link link_11.0_tip
- removed link link_12.0
- removed link link_13.0
- removed link link_14.0
- removed link link_15.0
- removed link link_15.0_tip
- removed link link_2.0
- removed link link_3.0
- removed link link_3.0_tip
- removed link link_4.0
- removed link link_5.0
- removed link link_6.0
- removed link link_7.0
- removed link link_7.0_tip
- removed link link_8.0
- removed link link_9.0
- added link link_0_0, mass 0.0119; collision box size=0.0196 0.0275 0.0164; visual mesh filename=meshes/allegro/link_0_0.obj
- added link link_10_0, mass 0.0355; collision box size=0.0196 0.0275 0.0384; visual mesh filename=meshes/allegro/link_2_0.obj
- added link link_11_0, mass 0.0096; collision sphere radius=0.0001; visual mesh filename=meshes/allegro/link_3_0.obj
- added link link_11_0_tip, mass 0.0168; collision sphere radius=0.012; visual mesh filename=meshes/allegro/link_3_0_tip.obj
- added link link_12_0, mass 0.0176; collision box size=0.0358 0.034 0.0455; visual mesh filename=meshes/allegro/link_12_0_right.obj
- added link link_13_0, mass 0.0119; collision box size=0.0196 0.0275 0.0177; visual mesh filename=meshes/allegro/link_13_0.obj
- added link link_14_0, mass 0.038; collision box size=0.0196 0.0275 0.0514; visual mesh filename=meshes/allegro/link_14_0.obj
- added link link_15_0, mass 0.0388; collision sphere radius=0.0001; visual mesh filename=meshes/allegro/link_15_0.obj
- added link link_15_0_tip, mass 0.0168; collision sphere radius=0.012; visual mesh filename=meshes/allegro/link_15_0_tip.obj
- added link link_1_0, mass 0.065; collision box size=0.0196 0.0275 0.054; visual mesh filename=meshes/allegro/link_1_0.obj
- added link link_2_0, mass 0.0355; collision box size=0.0196 0.0275 0.0384; visual mesh filename=meshes/allegro/link_2_0.obj
- added link link_3_0, mass 0.0096; collision sphere radius=0.0001; visual mesh filename=meshes/allegro/link_3_0.obj
- added link link_3_0_tip, mass 0.0168; collision sphere radius=0.012; visual mesh filename=meshes/allegro/link_3_0_tip.obj
- added link link_4_0, mass 0.0119; collision box size=0.0196 0.0275 0.0164; visual mesh filename=meshes/allegro/link_0_0.obj
- added link link_5_0, mass 0.065; collision box size=0.0196 0.0275 0.054; visual mesh filename=meshes/allegro/link_1_0.obj
- added link link_6_0, mass 0.0355; collision box size=0.0196 0.0275 0.0384; visual mesh filename=meshes/allegro/link_2_0.obj
- added link link_7_0, mass 0.0096; collision sphere radius=0.0001; visual mesh filename=meshes/allegro/link_3_0.obj
- added link link_7_0_tip, mass 0.0168; collision sphere radius=0.012; visual mesh filename=meshes/allegro/link_3_0_tip.obj
- added link link_8_0, mass 0.0119; collision box size=0.0196 0.0275 0.0164; visual mesh filename=meshes/allegro/link_0_0.obj
- added link link_9_0, mass 0.065; collision box size=0.0196 0.0275 0.054; visual mesh filename=meshes/allegro/link_1_0.obj
- link base_link: geometry collision box size=0.01 0.01 0.01; visual mesh filename=meshes/allegro/base_link.obj
Joints:
- removed joint joint_0.0
- removed joint joint_1.0
- removed joint joint_10.0
- removed joint joint_11.0
- removed joint joint_11.0_tip
- removed joint joint_12.0
- removed joint joint_13.0
- removed joint joint_14.0
- removed joint joint_15.0
- removed joint joint_15.0_tip
- removed joint joint_2.0
- removed joint joint_3.0
- removed joint joint_3.0_tip
- removed joint joint_4.0
- removed joint joint_5.0
- removed joint joint_6.0
- removed joint joint_7.0
- removed joint joint_7.0_tip
- removed joint joint_8.0
- removed joint joint_9.0
- added joint joint_0_0: type revolute, parent base_link, child link_0_0, origin xyz=0 0.0435 -0.001542 rpy=-0.08726646255 0 0, axis 0 0 1, limit lower=-0.47 upper=0.47 effort=0.35 velocity=6.283
- added joint joint_10_0: type revolute, parent link_9_0, child link_10_0, origin xyz=0 0 0.054, axis 0 1 0, limit lower=-0.174 upper=1.709 effort=0.35 velocity=6.283
- added joint joint_11_0: type revolute, parent link_10_0, child link_11_0, origin xyz=0 0 0.0384, axis 0 1 0, limit lower=-0.227 upper=1.618 effort=0.35 velocity=6.283
- added joint joint_11_0_tip: type fixed, parent link_11_0, child link_11_0_tip, origin xyz=0 0 0.0267 rpy=0 0 0
- added joint joint_12_0: type revolute, parent base_link, child link_12_0, origin xyz=-0.0182 0.019333 -0.045987 rpy=0 -1.65806278845 -1.5707963259, axis -1 0 0, limit lower=0.263 upper=1.396 effort=0.35 velocity=6.283
- added joint joint_13_0: type revolute, parent link_12_0, child link_13_0, origin xyz=-0.027 0.005 0.0399, axis 0 0 1, limit lower=-0.105 upper=1.163 effort=0.35 velocity=6.283
- added joint joint_14_0: type revolute, parent link_13_0, child link_14_0, origin xyz=0 0 0.0177, axis 0 1 0, limit lower=-0.189 upper=1.644 effort=0.35 velocity=6.283
- added joint joint_15_0: type revolute, parent link_14_0, child link_15_0, origin xyz=0 0 0.0514, axis 0 1 0, limit lower=-0.162 upper=1.719 effort=0.35 velocity=6.283
- added joint joint_15_0_tip: type fixed, parent link_15_0, child link_15_0_tip, origin xyz=0 0 0.0423 rpy=0 0 0
- added joint joint_1_0: type revolute, parent link_0_0, child link_1_0, origin xyz=0 0 0.0164, axis 0 1 0, limit lower=-0.196 upper=1.61 effort=0.35 velocity=6.283
- added joint joint_2_0: type revolute, parent link_1_0, child link_2_0, origin xyz=0 0 0.054, axis 0 1 0, limit lower=-0.174 upper=1.709 effort=0.35 velocity=6.283
- added joint joint_3_0: type revolute, parent link_2_0, child link_3_0, origin xyz=0 0 0.0384, axis 0 1 0, limit lower=-0.227 upper=1.618 effort=0.35 velocity=6.283
- added joint joint_3_0_tip: type fixed, parent link_3_0, child link_3_0_tip, origin xyz=0 0 0.0267 rpy=0 0 0
- added joint joint_4_0: type revolute, parent base_link, child link_4_0, origin xyz=0 0 0.0007 rpy=0.0 0 0, axis 0 0 1, limit lower=-0.47 upper=0.47 effort=0.35 velocity=6.283
- added joint joint_5_0: type revolute, parent link_4_0, child link_5_0, origin xyz=0 0 0.0164, axis 0 1 0, limit lower=-0.196 upper=1.61 effort=0.35 velocity=6.283
- added joint joint_6_0: type revolute, parent link_5_0, child link_6_0, origin xyz=0 0 0.054, axis 0 1 0, limit lower=-0.174 upper=1.709 effort=0.35 velocity=6.283
- added joint joint_7_0: type revolute, parent link_6_0, child link_7_0, origin xyz=0 0 0.0384, axis 0 1 0, limit lower=-0.227 upper=1.618 effort=0.35 velocity=6.283
- added joint joint_7_0_tip: type fixed, parent link_7_0, child link_7_0_tip, origin xyz=0 0 0.0267 rpy=0 0 0
- added joint joint_8_0: type revolute, parent base_link, child link_8_0, origin xyz=0 -0.0435 -0.001542 rpy=0.08726646255 0 0, axis 0 0 1, limit lower=-0.47 upper=0.47 effort=0.35 velocity=6.283
- added joint joint_9_0: type revolute, parent link_8_0, child link_9_0, origin xyz=0 0 0.0164, axis 0 1 0, limit lower=-0.196 upper=1.61 effort=0.35 velocity=6.283

File: assets/allegro/allegro_internal.urdf (robot description, URDF)
Before this commit: robot allegro_hand_right, 21 links, 20 joints
Links:
- removed link link_0.0
- removed link link_1.0
- removed link link_10.0
- removed link link_11.0
- removed link link_11.0_tip
- removed link link_12.0
- removed link link_13.0
- removed link link_14.0
- removed link link_15.0
- removed link link_15.0_tip
- removed link link_2.0
- removed link link_3.0
- removed link link_3.0_tip
- removed link link_4.0
- removed link link_5.0
- removed link link_6.0
- removed link link_7.0
- removed link link_7.0_tip
- removed link link_8.0
- removed link link_9.0
- added link link_0_0, mass 0.0119; collision box size=0.0196 0.0275 0.0164; visual mesh filename=meshes/allegro/link_0_0.obj
- added link link_10_0, mass 0.0355; collision box size=0.0196 0.0275 0.0384; visual mesh filename=meshes/allegro/link_2_0.obj
- added link link_11_0, mass 0.0096; collision sphere radius=0.0001; visual mesh filename=meshes/allegro/link_3_0.obj
- added link link_11_0_tip, mass 0.0168; collision sphere radius=0.01235; visual mesh filename=meshes/allegro/digitv2.obj
- added link link_12_0, mass 0.0176; collision box size=0.0358 0.034 0.0455; visual mesh filename=meshes/allegro/link_12_0_right.obj
- added link link_13_0, mass 0.0119; collision box size=0.0196 0.0275 0.0177; visual mesh filename=meshes/allegro/link_13_0.obj
- added link link_14_0, mass 0.038; collision box size=0.0196 0.0275 0.0514; visual mesh filename=meshes/allegro/link_14_0.obj
- added link link_15_0, mass 0.0388; collision sphere radius=0.0001; visual mesh filename=meshes/allegro/link_15_0.obj
- added link link_15_0_tip, mass 0.0168; collision sphere radius=0.01235; visual mesh filename=meshes/allegro/digitv2.obj
- added link link_1_0, mass 0.065; collision box size=0.0196 0.0275 0.054; visual mesh filename=meshes/allegro/link_1_0.obj
- added link link_2_0, mass 0.0355; collision box size=0.0196 0.0275 0.0384; visual mesh filename=meshes/allegro/link_2_0.obj
- added link link_3_0, mass 0.0096; collision sphere radius=0.0001; visual mesh filename=meshes/allegro/link_3_0.obj
- added link link_3_0_tip, mass 0.0168; collision sphere radius=0.01235; visual mesh filename=meshes/allegro/digitv2.obj
- added link link_4_0, mass 0.0119; collision box size=0.0196 0.0275 0.0164; visual mesh filename=meshes/allegro/link_0_0.obj
- added link link_5_0, mass 0.065; collision box size=0.0196 0.0275 0.054; visual mesh filename=meshes/allegro/link_1_0.obj
- added link link_6_0, mass 0.0355; collision box size=0.0196 0.0275 0.0384; visual mesh filename=meshes/allegro/link_2_0.obj
- added link link_7_0, mass 0.0096; collision sphere radius=0.0001; visual mesh filename=meshes/allegro/link_3_0.obj
- added link link_7_0_tip, mass 0.0168; collision sphere radius=0.01235; visual mesh filename=meshes/allegro/digitv2.obj
- added link link_8_0, mass 0.0119; collision box size=0.0196 0.0275 0.0164; visual mesh filename=meshes/allegro/link_0_0.obj
- added link link_9_0, mass 0.065; collision box size=0.0196 0.0275 0.054; visual mesh filename=meshes/allegro/link_1_0.obj
- link base_link: geometry collision box size=0.01 0.01 0.01; visual mesh filename=meshes/allegro/base_link.obj
Joints:
- removed joint joint_0.0
- removed joint joint_1.0
- removed joint joint_10.0
- removed joint joint_11.0
- removed joint joint_11.0_tip
- removed joint joint_12.0
- removed joint joint_13.0
- removed joint joint_14.0
- removed joint joint_15.0
- removed joint joint_15.0_tip
- removed joint joint_2.0
- removed joint joint_3.0
- removed joint joint_3.0_tip
- removed joint joint_4.0
- removed joint joint_5.0
- removed joint joint_6.0
- removed joint joint_7.0
- removed joint joint_7.0_tip
- removed joint joint_8.0
- removed joint joint_9.0
- added joint joint_0_0: type revolute, parent base_link, child link_0_0, origin xyz=0 0.0435 -0.001542 rpy=-0.08726646255 0 0, axis 0 0 1, limit lower=-0.47 upper=0.47 effort=0.35 velocity=6.283
- added joint joint_10_0: type revolute, parent link_9_0, child link_10_0, origin xyz=0 0 0.054, axis 0 1 0, limit lower=-0.174 upper=1.709 effort=0.35 velocity=6.283
- added joint joint_11_0: type revolute, parent link_10_0, child link_11_0, origin xyz=0 0 0.0384, axis 0 1 0, limit lower=-0.227 upper=1.618 effort=0.35 velocity=6.283
- added joint joint_11_0_tip: type fixed, parent link_11_0, child link_11_0_tip, origin xyz=0 0 0.0147 rpy=0 0 0
- added joint joint_12_0: type revolute, parent base_link, child link_12_0, origin xyz=-0.0182 0.019333 -0.045987 rpy=0 -1.65806278845 -1.5707963259, axis -1 0 0, limit lower=0.263 upper=1.396 effort=0.35 velocity=6.283
- added joint joint_13_0: type revolute, parent link_12_0, child link_13_0, origin xyz=-0.027 0.005 0.0399, axis 0 0 1, limit lower=-0.105 upper=1.163 effort=0.35 velocity=6.283
- added joint joint_14_0: type revolute, parent link_13_0, child link_14_0, origin xyz=0 0 0.0177, axis 0 1 0, limit lower=-0.189 upper=1.644 effort=0.35 velocity=6.283
- added joint joint_15_0: type revolute, parent link_14_0, child link_15_0, origin xyz=0 0 0.0514, axis 0 1 0, limit lower=-0.162 upper=1.719 effort=0.35 velocity=6.283
- added joint joint_15_0_tip: type fixed, parent link_15_0, child link_15_0_tip, origin xyz=0 0 0.0303 rpy=0 0 0
- added joint joint_1_0: type revolute, parent link_0_0, child link_1_0, origin xyz=0 0 0.0164, axis 0 1 0, limit lower=-0.196 upper=1.61 effort=0.35 velocity=6.283
- added joint joint_2_0: type revolute, parent link_1_0, child link_2_0, origin xyz=0 0 0.054, axis 0 1 0, limit lower=-0.174 upper=1.709 effort=0.35 velocity=6.283
- added joint joint_3_0: type revolute, parent link_2_0, child link_3_0, origin xyz=0 0 0.0384, axis 0 1 0, limit lower=-0.227 upper=1.618 effort=0.35 velocity=6.283
- added joint joint_3_0_tip: type fixed, parent link_3_0, child link_3_0_tip, origin xyz=0 0 0.0147 rpy=0 0 0
- added joint joint_4_0: type revolute, parent base_link, child link_4_0, origin xyz=0 0 0.0007 rpy=0.0 0 0, axis 0 0 1, limit lower=-0.47 upper=0.47 effort=0.35 velocity=6.283
- added joint joint_5_0: type revolute, parent link_4_0, child link_5_0, origin xyz=0 0 0.0164, axis 0 1 0, limit lower=-0.196 upper=1.61 effort=0.35 velocity=6.283
- added joint joint_6_0: type revolute, parent link_5_0, child link_6_0, origin xyz=0 0 0.054, axis 0 1 0, limit lower=-0.174 upper=1.709 effort=0.35 velocity=6.283
- added joint joint_7_0: type revolute, parent link_6_0, child link_7_0, origin xyz=0 0 0.0384, axis 0 1 0, limit lower=-0.227 upper=1.618 effort=0.35 velocity=6.283
- added joint joint_7_0_tip: type fixed, parent link_7_0, child link_7_0_tip, origin xyz=0 0 0.0147 rpy=0 0 0
- added joint joint_8_0: type revolute, parent base_link, child link_8_0, origin xyz=0 -0.0435 -0.001542 rpy=0.08726646255 0 0, axis 0 0 1, limit lower=-0.47 upper=0.47 effort=0.35 velocity=6.283
- added joint joint_9_0: type revolute, parent link_8_0, child link_9_0, origin xyz=0 0 0.0164, axis 0 1 0, limit lower=-0.196 upper=1.61 effort=0.35 velocity=6.283
